Commit message: change

File: crane_x7_description/urdf/crane_x7.urdf.xacro (robot description, xacro)
@@ -22,14 +22,14 @@
        right-handed robots. -->
   <crane_x7 parent="base_link"
-              base_color="red"
-              shoulder_color="white"
-              shoulder_joint_cover_color="red"
-              upper_arm_upper_color="white"
-              upper_arm_lower_color="white"
-              elbow_joint_cover_color="red"
-              lower_arm_upper_color="white"
+              base_color="white"
+              shoulder_color="blue"
+              shoulder_joint_cover_color="white"
+              upper_arm_upper_color="blue"
+              upper_arm_lower_color="blue"
+              elbow_joint_cover_color="white"
+              lower_arm_upper_color="blue"
               lower_arm_lower_color="white"
               wrist_color="white"
-              hand_color="red"
+              hand_color="white"
               joints_vlimit="4.81710873"
               shoulder_llimit="-2.97132"

File: crane_x7_description/urdf/crane_x7.xacro (robot description, xacro)
@@ -4,4 +4,5 @@
   <xacro:include filename="$(find crane_x7_description)/urdf/crane_x7_arm.xacro"/>
   <xacro:include filename="$(find crane_x7_description)/urdf/crane_x7_wide_two_finger_gripper.xacro"/>
+  <xacro:include filename="$(find crane_x7_description)/urdf/camera.urdf"/>
   <material name="black">
     <color rgba="0.2 0.2 0.2 1.0"/>

File: crane_x7_description/urdf/crane_x7_arm.xacro (robot description, xacro)
@@ -485,20 +485,20 @@
     </gazebo>
     <gazebo reference="${NAME_LINK_BASE}">
-      <material>Gazebo/Red</material>
+      <material>Gazebo/White</material>
     </gazebo>
     <gazebo reference="${NAME_LINK_1}">
-      <material>Gazebo/White</material>
+      <material>Gazebo/Blue</material>
     </gazebo>
     <gazebo reference="${NAME_LINK_2}">
-      <material>Gazebo/White</material>
+      <material>Gazebo/Blue</material>
     </gazebo>
     <gazebo reference="${NAME_LINK_3}">
-      <material>Gazebo/White</material>
+      <material>Gazebo/Blue</material>
     </gazebo>
     <gazebo reference="${NAME_LINK_4}">
-      <material>Gazebo/White</material>
+      <material>Gazebo/Blue</material>
     </gazebo>
     <gazebo reference="${NAME_LINK_5}">
-      <material>Gazebo/White</material>
+      <material>Gazebo/Blue</material>
     </gazebo>
     <gazebo reference="${NAME_LINK_6}">
@@ -506,14 +506,14 @@
     </gazebo>
     <gazebo reference="${NAME_LINK_COVER_2_L}">
-      <material>Gazebo/Red</material>
+      <material>Gazebo/White</material>
     </gazebo>
     <gazebo reference="${NAME_LINK_COVER_2_R}">
-      <material>Gazebo/Red</material>
+      <material>Gazebo/White</material>
     </gazebo>
     <gazebo reference="${NAME_LINK_COVER_4_L}">
-      <material>Gazebo/Red</material>
+      <material>Gazebo/White</material>
     </gazebo>
     <gazebo reference="${NAME_LINK_COVER_4_R}">
-      <material>Gazebo/Red</material>
+      <material>Gazebo/White</material>
     </gazebo>
   </xacro:macro>

File: crane_x7_description/urdf/crane_x7_wide_two_finger_gripper.xacro (robot description, xacro)
@@ -128,15 +128,15 @@
     </gazebo>
     <gazebo reference="${name}_base_link">
-      <material>Gazebo/Red</material>
+      <material>Gazebo/Blue</material>
     </gazebo>
     <gazebo reference="${name}_finger_a_link">
       <mu1>0.8</mu1>
       <mu2>0.8</mu2>
-      <material>Gazebo/Red</material>
+      <material>Gazebo/Blue</material>
     </gazebo>
     <gazebo reference="${name}_finger_b_link">
       <mu1>0.8</mu1>
       <mu2>0.8</mu2>
-      <material>Gazebo/Red</material>
+      <material>Gazebo/Blue</material>
     </gazebo>
   </xacro:macro>
